File: pcb/il-flatto/internals.kicad_sch (KiCad schematic)
At the start: 35 parts, among them J100 USB_C_Receptacle_USB2.0, SW100 CHRG_CURR, SW101 CHRG_EN, SW102 PWR SEL, SW103 SW_SPST, U100 MCP73831-2-MC, U101 NCV8605MN33T2G, U102 ATmega1284P-M, Y100 12MHz

Commit message: good to go?
Parts:
- removed SW100: CHRG_CURR, symbol Switch:SW_DPDT_x2
- removed SW101: CHRG_EN, symbol Switch:SW_DPDT_x2
- removed Y100: 12MHz, symbol Device:Crystal_Small
- added D101: LED, LED_SMD:LED_0603_1608Metric, symbol Device:LED
- added J103: ISP, footprints:PinSocket_2x03_P2.54mm zero footprint mirror, symbol Connector_Generic:Conn_02x03_Odd_Even
- added J105: JTAG, footprints:PinSocket_2x05_P2.54mm zero footprint mirror, symbol Connector_Generic:Conn_02x05_Odd_Even
- added JP103: Conn_01x03, footprints:PinHeader_1x03_P2.54mm zero footprint, symbol Connector_Generic:Conn_01x03
- added Q101: 12MHz, Crystal:Crystal_SMD_Abracon_ABM8G-4Pin_3.2x2.5mm, symbol Device:Crystal_GND24_Small
- added R104: 220, Resistor_SMD:R_0402_1005Metric, symbol Device:R
- added R106, R107, R108, R109, R110, R111: 68, Resistor_SMD:R_0402_1005Metric, symbol Device:R
- added S103: SW_DPST_x2, footprints:CVS-02TB mirrored, symbol Switch:SW_DPST_x2
- added X102: SD_Card, symbol Connector:SD_Card
- added X103: BAT, Connector_JST:JST_PH_B2B-PH-K_1x02_P2.00mm_Vertical, symbol Connector_Generic:Conn_01x02
- C101: renamed from C103; footprint (none) -> Capacitor_SMD:C_0402_1005Metric
- C102: renamed from C104; footprint (none) -> Capacitor_SMD:C_0402_1005Metric
- C103: renamed from C106; footprint (none) -> Capacitor_SMD:C_0402_1005Metric
- C104: renamed from C101; footprint (none) -> Capacitor_SMD:C_0402_1005Metric
- C106: renamed from C102; footprint (none) -> Capacitor_SMD:C_0402_1005Metric
- C107: renamed from C108; footprint (none) -> Capacitor_SMD:C_0402_1005Metric
- C108: renamed from C109; footprint (none) -> Capacitor_SMD:C_0402_1005Metric
- C109: renamed from C110; footprint (none) -> Capacitor_SMD:C_0402_1005Metric
- C110: renamed from C111; footprint (none) -> Capacitor_SMD:C_0402_1005Metric
- C111: renamed from C112; footprint (none) -> Capacitor_SMD:C_0402_1005Metric
- C112: renamed from C113; footprint (none) -> Capacitor_SMD:C_0402_1005Metric
- C113: renamed from C115; footprint (none) -> Capacitor_SMD:C_0402_1005Metric
- C114: footprint (none) -> Capacitor_SMD:C_0402_1005Metric
- C205: renamed from C107; footprint (none) -> Capacitor_SMD:C_0402_1005Metric
- C206: renamed from C105; footprint (none) -> Capacitor_SMD:C_0402_1005Metric
- D102: renamed from D100; footprint (none) -> LED_SMD:LED_0603_1608Metric
- R102: renamed from R106; footprint (none) -> Resistor_SMD:R_0402_1005Metric
- R103: renamed from R104; footprint (none) -> Resistor_SMD:R_0402_1005Metric
- R105: renamed from R109; footprint (none) -> Resistor_SMD:R_0402_1005Metric
- R112: renamed from R107; footprint (none) -> Resistor_SMD:R_0402_1005Metric
- R201: renamed from R102; footprint (none) -> Resistor_SMD:R_0402_1005Metric
- R202: renamed from R103; footprint (none) -> Resistor_SMD:R_0402_1005Metric
- R203: renamed from R100; value 2k -> 2.5k; footprint (none) -> Resistor_SMD:R_0402_1005Metric
- R204: renamed from R101; footprint (none) -> Resistor_SMD:R_0402_1005Metric
- S101: renamed from SW102; value PWR SEL -> S1
- S102: renamed from SW103; footprint (none) -> footprints:SW_TL3780AF240QG
- X101: renamed from J100; footprint (none) -> footprints:GCT_USB4110-GF-A_REVB
- renumbered C100 to C105, R105 to R101, U102 to U101, U101 to U102, U100 to U103
Connections:
- net GND: now also X101.A1/B12 (GND), X101.B1/A12 (GND), X101.S2 (SHIELD), X101.S3 (SHIELD), X101.S4 (SHIELD), J103.6 (Pin_6), J105.10 (Pin_10), J105.2 (Pin_2), Q101.2, Q101.4, R104.2, S103.3 (A), X102.12 (SHELL1), X102.13 (SHELL2), X102.3 (VSS), X102.6 (VSS), X103.2 (Pin_2); no longer R203.2, R204.2, X101.A1 (GND), X101.A12 (GND), X101.B1 (GND), X101.B12 (GND)
- net PB0: now also R110.1
- net PB1: now also R111.2
- net PB2: now also R101.1; no longer R102.1
- net PB3: now also R102.2; no longer R101.2
- net PB4: now also R106.1
- net PB5: now also J103.4 (Pin_4), R107.2
- net PB6: now also J103.1 (Pin_1), R109.2
- net PB7: now also J103.3 (Pin_3), JP103.3 (Pin_3), R108.2
- net PC2: now also J105.1 (Pin_1)
- net PC3: now also J105.5 (Pin_5)
- net PC4: now also J105.3 (Pin_3)
- net PC5: now also J105.9 (Pin_9)
- net Q1_1: now also Q101.1
- net Q1_2: now also Q101.3
- net VBUS: now also C104.2, X101.A4/B9 (VBUS), X101.B4/A9 (VBUS); no longer X101.A4 (VBUS), X101.A9 (VBUS), X101.B4 (VBUS), X101.B9 (VBUS)
- net VDD: now also J103.2 (Pin_2), J105.4 (Pin_4), J105.7 (Pin_7), JP103.1 (Pin_1), X102.4 (VDD)
- net V_BAT: now also X103.1 (Pin_1)
- net n_reset: now also J103.5 (Pin_5), J105.6 (Pin_6)
- net USB D-: now reaches R103.2, X101.A7 (D-), X101.B7 (D-)
- net USB D-: now also R102.1; no longer R101.1
- net LDO_in: now reaches S101.2 (B), U102.1 (VIN), U102.3 (NC/EN), U102.6 (VIN)
- net LDO_in: no longer C104.2
- net USB D+: now reaches X101.A6 (D+), X101.B6 (D+)
- net USB D+: now also R101.2; no longer R102.2
- net at R204.1: now also R203.1, U103.8 (PROG)
- new net: D101.1 (K), R104.1
- new net: D101.2 (A), JP103.2 (Pin_2)
- new net: R111.1, X102.10 (CARD_DETECT)
- new net: R110.2, X102.11 (WRITE_PROTECT)
- new net: R204.2, S103.2 (B), S103.4 (B)
- new net: R106.2, X102.1 (CD/DAT3)
- new net: R107.1, X102.2 (CMD)
- new net: R108.1, X102.5 (CLK)
- new net: R109.1, X102.7 (DAT0)
- new net: R203.2, S103.1 (A)
- no-connect marks 3 -> 5
Other:
- added sheet Row1 (LED_ROW.kicad_sch)
- added sheet Row2 (LED_ROW.kicad_sch)
- added sheet Row3 (LED_ROW.kicad_sch)
- added sheet Row4 (LED_ROW.kicad_sch)
- added sheet Row5 (LED_ROW.kicad_sch)
- added sheet Row6 (LED_ROW.kicad_sch)
- added sheet Row7 (LED_ROW.kicad_sch)
- added sheet Row8 (LED_ROW.kicad_sch)
- note added: "Connectors"
- note added: "LEDs"
- note added: "]Pwr ]Usr"
- note added: "closed: 500mA open: 100mA"
- note added: "closed: ON open: OFF"
- note removed: "100mA"
- note removed: "500mA"
- note removed: "OFF"
- note removed: "ON"
- moved on the sheet: C101, C102, C104, R101, R102, R105, R203, R204, S102
