File: pcb/il-flatto/outer layers.kicad_sch (KiCad schematic)
At the start: 45 parts, among them IC1 ATmega1284P-P, IC2 MCP1825S, IC3 MAX1811, J3 ISP, J4 SD_Card, J5 JTAG, Q1 12MHz, SW4 SW_SPST, X1 USB_B_Mini, X3 BAT

Commit message: good to go?
Parts:
- S1: renamed from Se100; value PWR SEL -> S1
- S3: footprint footprints:SW_CAS-D20TA -> footprints:CAS-D20TB
- X2: renamed from J4; footprint (none) -> footprints:sd card
- renumbered SW4 to S2
Connections:
- net LDO_in: now reaches IC2.1 (VI), S1.2 (B)
- net USB+ renamed USB D+
- net USB- renamed USB D-
Other:
- moved on the sheet: R1, R2, R3
